File: pcbs/jabr-control-v1/mipi-connectors.kicad_sch (KiCad schematic)
At the start: 5 parts, among them J1501 FH12-22S-0.5SH, J1502 FH12-22S-0.5SH

Commit message: Updated FH12-22S-0.5SH footprints
Parts:
- J1501, J1502: footprint project_footprints:FH12-22S-0.5SH -> project_footprints:Hirose_FH12-22S-0.5SH_1x22-1MP_P0.50mm_Horizontal
Changed lines of the file:
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@@
 			)
 		)
-		(property "Footprint" "project_footprints:FH12-22S-0.5SH"
+		(property "Footprint" "project_footprints:Hirose_FH12-22S-0.5SH_1x22-1MP_P0.50mm_Horizontal"
 			(at 181.61 132.08 0)
 			(effects
@@
 			)
 		)
-		(property "Footprint" "project_footprints:FH12-22S-0.5SH"
+		(property "Footprint" "project_footprints:Hirose_FH12-22S-0.5SH_1x22-1MP_P0.50mm_Horizontal"
 			(at 72.39 132.08 0)
 			(effects
