File: pcbs/jabr-control-v1/m-2-e-key.kicad_sch (KiCad schematic)
At the start: 12 parts, among them J4001 MDT320E0X001, J401 U.FL-R-SMT-K_895, J402 U.FL-R-SMT-K_895, Y401 ASEK-32.768KHZ-LRT

Commit message: Added v2 project
Parts:
- removed AE401, AE402: EMPCB.SMAFSTJ.B.HT, project_footprints:sma_edge_mount, symbol RF-CONN:EMPCB.SMAFSTJ.B.HT
- removed J401, J402: U.FL-R-SMT-K_895, project_footprints:UFLRSMTK895, symbol RF-CONN:U.FL-R-SMT-K_895
Other:
- note removed: "U.FL to SMA converters"
