File: pcbs/jabrj-control-v2/m-2-e-key.kicad_sch (KiCad schematic)
At the start: 5 parts, among them J1201 MDT420E0X001, Y1201 ASEK-32.768KHZ-LRT

Commit message: Layout started
Connections:
- net GND: now also J1201.MP1, J1201.MP2
