File: pcbs/jabrj-control-v2/jabrj-control-v2.kicad_pcb (KiCad board)
At the start: 6 copper layers, 70 x 80 mm, 315 parts, among them J1101 MSPE-J2L0-x00, J1201 MDT420E0X001, J301 43045-0201, J701 FFC3A20-05-G, J702 JST-SH-4-Vertical, J801 48406-0003, J802 ARJM11D7-502-AB-EW2, J803 TYPE-C-31-M-12, J804 FH12-20S-0.5SH, J805 FH12-20S-0.5SH, J901 FH12-22S-0.5SH, J902 FH12-22S-0.5SH, Q401 DMN21D2UFB-7B, Q402 DMN21D2UFB-7B, Q403 DMN21D2UFB-7B, Q701 DMN21D2UFB-7B, SW701 TS20-42-25-WT-160-SMT-TR, U1001 SYA75603A, U1002 PCI11010C, U1003 AT24C64D-MAHM-E, U1101 LAN8870, U301 TVS3301DRBR, U302 TPS26600RHFR, U401 AZV3001FZ4-7, U402 TPS259472ARPWR, U403 MAX20008AFOC/VY+T, U501 TPS7B8133QDRVRQ1, U502 TPS2116DRL, U601 TPS22991CNRAAR, U602 TPS62827DMQR, U603 TPS62825DMQR, U701 PESD4USB3BTTS-QX, U702 NX3DV221GM, U801 PESD4USB3BTTS-QX, U802 PESD4USB3BTTS-QX, U803 PESD4USB3BTTS-QX, U804 PESD4USB3BTTS-QX, U805 PESD4USB3BTTS-QX, U806 AP22653FDZ-7, U807 PESD4USB3BTTS-QX, Y1001 XRCGB25M000F3A16R0, Y1101 XRCGB25M000F3A16R0, Y1201 ASEK-32.768KHZ-LRT

Commit message: Layout almost done
Parts:
- added D403: RED, project_footprints:C_0402, F.Cu at (100.6, 71.7)
- added D404: RED, project_footprints:C_0402, F.Cu at (100.6, 73.7)
- C1001, C1002, C1003, C1004, C1005, C1006, C1007, C1008, C1009, C1010, C1011, C1012, C1013, C1014, C1019, C1020, C1021, C1022, C1023, C1024, C1025, C1026, C1027, C1028, C1029, C1030, C1031, C1032, C1033, C1034, C1035, C1036, C1037, C1038, C1039, C1040, C1041, C1042, C1043, C1044, C1045, C1046, C1047, C1051, C1101, C1102, C1103, C1104, C1105, C1106, C1107, C1108, C1109, C1110, C1111, C1112, C1113, C1114, C1115, C1116, C1117, C1118, C1119, C1120, C1123, C901, C902, D1101, D704, D705, R1003, R1004, R1005, R1006, R1008, R1009, R1010, R1011, R1012, R1013, R1014, R1015, R1016, R1017, R1018, R1019, R1020, R1021, R1022, R1023, R1024, R1025, R1101, R1102, R1103, R1104, R1105, R1106, R1107, R1108, R1109, R1110, R1111, R1112, R1113, R1114, R1115, R1116, R1117, R413, R414, R703, R704, R901, R902, R903, TP1001, TP1002, TP1003, TP1004, TP1007, TP1102, TP1103, TP1104, TP1105, TP1106, TP402: moved to B.Cu
- C1048, C1049: moved to F.Cu
- moved D1101 148.6 mm to (192.0, 62.0), turned to 180 degrees
- moved C1051 143.8 mm to (205.5, 93.6)
- moved D1001 137.5 mm to (190.8, 78.4), turned to 90 degrees
- moved R1025 134.2 mm to (205.5, 94.8)
- moved TP1004 126.7 mm to (192.6, 78.7)
- moved R1001 126.6 mm to (192.2, 78.5), turned to -90 degrees
- moved TP1001 124.7 mm to (190.1, 78.7)
- moved R1007 124.6 mm to (190.2, 92.8)
- moved C1005 121.9 mm to (170.0, 81.8)
- moved R1016 121.8 mm to (158.6, 72.0), turned to 90 degrees
- moved C1009 121.6 mm to (170.0, 82.8)
- moved R1015 119.7 mm to (157.6, 72.0), turned to 90 degrees
- moved C1012 119.7 mm to (170.0, 85.2)
- moved C1014 119.4 mm to (170.0, 86.2)
- moved TP1103 118.5 mm to (167.0, 96.2)
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Connections:
- net /MIPI Connectors/~{MIPI1_RST} renamed /MIPI Connectors/MIPI1_PWR_EN
- J1201 pad MP1: (no net) -> GND
- J1201 pad MP2: (no net) -> GND
- J901 pad MP1: (no net) -> unconnected-(J901-PadMP1)
- J901 pad MP2: (no net) -> unconnected-(J901-PadMP2)
- J902 pad MP1: (no net) -> unconnected-(J902-PadMP1)
- J902 pad MP2: (no net) -> unconnected-(J902-PadMP2)
- TP702 pad 1: /CM5/DP -> /CM5/USB2_DEV.DP
- TP703 pad 1: /CM5/DN -> /CM5/USB2_DEV.DN
- U807 pad 2: /CM5/USB2_DEV.CC1 -> /CM5/USB2_DEV.DP
- U807 pad 5: /CM5/USB2_DEV.DP -> /CM5/USB2_DEV.CC1
- U807 pad 6: /CM5/USB2_DEV.DP -> /CM5/USB2_DEV.CC1
- U807 pad 9: /CM5/USB2_DEV.CC1 -> /CM5/USB2_DEV.DP
Routing:
- net /1000BASE-T1 PHY/MDIO: track 0.00 -> 5.77 mm
- net /1000BASE-T1 PHY/MDC: track 0.00 -> 5.53 mm
- net /M.2 E-Key/M2_SPI.CS: track 0.00 -> 5.28 mm
- net /M.2 E-Key/M2_SPI.MOSI: track 0.00 -> 5.26 mm
- net /M.2 E-Key/M2_SPI.MISO: track 0.00 -> 5.22 mm
- net /M.2 E-Key/M2_SPI.CLK: track 0.00 -> 5.01 mm
- net /M.2 E-Key/M2_SPI.~{INT}: track 0.00 -> 4.84 mm
