File: pcbs/jabrj-control-v2/jabrj-control-v2.kicad_pcb (KiCad board)
At the start: 6 copper layers, 70 x 80 mm, 317 parts, among them J1101 MSPE-J2L0-x00, J1201 MDT420E0X001, J301 43045-0201, J701 FFC3A20-05-G, J702 JST-SH-4-Vertical, J801 48406-0003, J802 ARJM11D7-502-AB-EW2, J803 TYPE-C-31-M-12, J804 FH12-20S-0.5SH, J805 FH12-20S-0.5SH, J901 FH12-22S-0.5SH, J902 FH12-22S-0.5SH, Q401 DMN21D2UFB-7B, Q402 DMN21D2UFB-7B, Q403 DMN21D2UFB-7B, Q701 DMN21D2UFB-7B, SW701 TS20-42-25-WT-160-SMT-TR, U1001 SYA75603A, U1002 PCI11010C, U1003 AT24C64D-MAHM-E, U1101 LAN8870, U301 TVS3301DRBR, U302 TPS26600RHFR, U401 AZV3001FZ4-7, U402 TPS259472ARPWR, U403 MAX20008AFOC/VY+T, U501 TPS7B8133QDRVRQ1, U502 TPS2116DRL, U601 TPS22991CNRAAR, U602 TPS62827DMQR, U603 TPS62825DMQR, U701 PESD4USB3BTTS-QX, U702 NX3DV221GM, U801 PESD4USB3BTTS-QX, U802 PESD4USB3BTTS-QX, U803 PESD4USB3BTTS-QX, U804 PESD4USB3BTTS-QX, U805 PESD4USB3BTTS-QX, U806 AP22653FDZ-7, U807 PESD4USB3BTTS-QX, Y1001 XRCGB25M000F3A16R0, Y1101 XRCGB25M000F3A16R0, Y1201 ASEK-32.768KHZ-LRT

Commit message: 895 Unrouted
Parts:
- R1003: moved to F.Cu
- U301: value TVS3301DRBR -> TVS2701DRBR
- moved R1003 26.0 mm to (193.0, 92.1)
- moved C1052 4.00 mm to (159.6, 72.0), turned to 90 degrees
- moved C1053 4.00 mm to (163.6, 72.0)
- moved R1023 2.00 mm to (170.0, 75.9)
- moved C1027 1.41 mm to (170.5, 74.4)
- moved C1029 1.00 mm to (169.5, 74.4)
- moved C1031 1.00 mm to (171.5, 75.4), turned to -90 degrees
- moved C1014 0.71 mm to (169.5, 85.7), turned to -90 degrees
- moved C1012 0.71 mm to (170.5, 85.7), turned to -90 degrees
- moved C1005 0.71 mm to (170.5, 82.3), turned to 90 degrees
- moved C1009 0.71 mm to (169.5, 82.3), turned to 90 degrees
- moved C1048 0.28 mm to (174.0, 83.3)
- moved C1049 0.28 mm to (174.0, 82.3)
- moved TP1002 0.25 mm to (172.1, 82.3)
- moved U702 0.10 mm to (172.7, 80.2)
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Connections:
- C1017 pad 1: /PCIe Switch/P1_TXP -> /PCIe Switch/P1_TXN
- C1017 pad 2: /M.2 E-Key/TX_P -> /M.2 E-Key/TX_N
- C1018 pad 1: /PCIe Switch/P1_TXN -> /PCIe Switch/P1_TXP
- C1018 pad 2: /M.2 E-Key/TX_N -> /M.2 E-Key/TX_P
- U1001 pad 10: /M.2 E-Key/CLK_P -> /M.2 E-Key/CLK_N
- U1001 pad 11: /M.2 E-Key/CLK_N -> /M.2 E-Key/CLK_P
- U1002 pad 78: /M.2 E-Key/RX_P -> /M.2 E-Key/RX_N
- U1002 pad 79: /M.2 E-Key/RX_N -> /M.2 E-Key/RX_P
- U1002 pad 82: /PCIe Switch/P1_TXP -> /PCIe Switch/P1_TXN
- U1002 pad 83: /PCIe Switch/P1_TXN -> /PCIe Switch/P1_TXP
Routing:
- net /M.2 E-Key/RX_N: track 0.00 -> 27.0 mm, vias 0 -> 1
- net /M.2 E-Key/RX_P: track 0.00 -> 26.5 mm, vias 0 -> 1
- net /M.2 E-Key/CLK_N: track 0.00 -> 19.2 mm
- net /M.2 E-Key/CLK_P: track 0.00 -> 18.7 mm
- net /M.2 E-Key/TX_N: track 0.00 -> 18.3 mm, vias 0 -> 1
- net /M.2 E-Key/TX_P: track 0.00 -> 18.0 mm, vias 0 -> 1
- net /M.2 E-Key/M2_SPI.~{INT}: track 4.84 -> 20.1 mm, vias 0 -> 2
- net /M.2 E-Key/M2_SPI.MISO: track 5.22 -> 19.8 mm, vias 0 -> 1
- net /M.2 E-Key/M2_SPI.CS: track 5.28 -> 19.7 mm, vias 0 -> 2
- net /CM5/DP: track 0.00 -> 13.0 mm
- net /CM5/DN: track 0.00 -> 12.9 mm
- net /M.2 E-Key/M2_SPI.MOSI: track 5.26 -> 17.3 mm, vias 0 -> 1
- net /M.2 E-Key/M2_SPI.CLK: track 5.01 -> 15.6 mm, vias 0 -> 1
- net /CM5/RX_N: track 0.00 -> 9.41 mm, vias 0 -> 1
- net /CM5/RX_P: track 0.00 -> 9.41 mm, vias 0 -> 1
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- added copper zone on In1.Cu, net GND
- added copper zone on In4.Cu, net GND

Commit message: 651 Unrouted
Parts:
- removed R901: 2k2, project_footprints:R_0402
- added TP603: 1.5mm, project_footprints:TestPoint_Pad_D1.5mm, B.Cu at (148.9, 82.1)
- D705, R704: moved to F.Cu
- moved D705 72.4 mm to (196.3, 78.0), turned to 90 degrees
- moved TP1007 71.6 mm to (193.2, 73.5)
- moved R704 69.5 mm to (195.3, 78.0), turned to 90 degrees
- moved D704 65.7 mm to (196.3, 78.0), turned to 90 degrees
- moved R703 62.6 mm to (195.3, 78.0), turned to 90 degrees
- moved R1116 42.0 mm to (195.3, 73.5), turned to 90 degrees
- moved R1019 22.6 mm to (145.7, 72.8)
- moved R1021 21.2 mm to (145.7, 74.8)
- moved R1022 21.0 mm to (145.7, 73.8)
- moved U401 17.2 mm to (188.9, 109.8)
- moved D1101 12.3 mm to (196.3, 73.5), turned to 90 degrees
- moved R401 10.00 mm to (201.9, 112.7)
- moved R403 10.00 mm to (201.9, 108.7)
- moved R404 10.00 mm to (201.9, 106.8)
- moved D401 10.00 mm to (204.7, 112.5)
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Connections:
- J902 pad 17: /MIPI Connectors/MIPI1_PWR_EN -> /MIPI Connectors/CAM_GPIO2
Routing:
- net /CM5/MIPI0.D3_P: track 1.89 -> 49.5 mm, vias 0 -> 1
- net /CM5/MIPI0.D3_N: track 1.89 -> 49.1 mm, vias 0 -> 1
- net /CM5/MIPI0.D2_P: track 1.89 -> 47.0 mm, vias 0 -> 1
- net /CM5/MIPI0.D2_N: track 1.89 -> 46.6 mm, vias 0 -> 1
- net /CM5/MIPI0.CLK_P: track 1.89 -> 44.9 mm, vias 0 -> 1
- net /CM5/MIPI0.CLK_N: track 1.89 -> 44.5 mm, vias 0 -> 1
- net /CM5/MIPI0.D1_P: track 1.89 -> 42.8 mm, vias 0 -> 1
- net /CM5/MIPI0.D1_N: track 1.89 -> 42.4 mm, vias 0 -> 1
- net /1000BASE-T1 PHY/TX_CLK: track 0.00 -> 40.0 mm, vias 0 -> 2
- net /1000BASE-T1 PHY/TX_D2: track 0.00 -> 39.1 mm, vias 0 -> 2
- net /1000BASE-T1 PHY/TX_CTL: track 0.00 -> 39.0 mm, vias 0 -> 2
- net /1000BASE-T1 PHY/TX_D1: track 0.00 -> 39.0 mm, vias 0 -> 2
- net /1000BASE-T1 PHY/TX_D3: track 0.00 -> 38.8 mm, vias 0 -> 2
- net /1000BASE-T1 PHY/TX_D0: track 0.00 -> 38.7 mm, vias 0 -> 2
- net /1000BASE-T1 PHY/TRXN: track 0.00 -> 38.2 mm, vias 0 -> 2
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- added copper zone on B.Cu, net +1V1
- added copper zone on B.Cu, net +1V8_PCIE
- added copper zone on B.Cu, net +3V3_AON
- added copper zone on B.Cu, net +3V3_PCIE
- added copper zone on B.Cu, net GND
- added copper zone on F.Cu, net GND
Other:
- board text added: "DISK"
- board text added: "ON/OFF"
- board text added: "PWR"
- board text added: "SPE"
