File: pcbs/jabrj-control-v2/pcie-power.kicad_sch (KiCad schematic)
At the start: 32 parts, among them U601 TPS22991CNRAAR, U602 TPS62827DMQR, U603 TPS62825DMQR

Commit message: 651 Unrouted
Parts:
- added TP603: 1.5mm, project_footprints:TestPoint_Pad_D1.5mm, symbol Connector:TestPoint_Small
Connections:
- net +1V8_PCIE: now also TP603.1
