File: pcbs/jabrj-control-v2/power-in.kicad_sch (KiCad schematic)
At the start: 10 parts, among them J301 43045-0201, U301 TVS3301DRBR, U302 TPS26600RHFR

Commit message: 895 Unrouted
Parts:
- U301: value TVS3301DRBR -> TVS2701DRBR; symbol SURGE:TVS3301DRBR -> SURGE:TVS2701DRBR; Height (none) -> 1; Manufacturer_Name (none) -> Texas Instruments; Manufacturer_Part_Number (none) -> TVS2701DRBR; Mouser Part Number (none) -> 595-TVS2701DRBR; Mouser Price/Stock (none) -> https://www.mouser.co.uk/ProductDetail/Texas-Instruments/TV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
Changed lines of the file:
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@@
 	)
 	(symbol
-		(lib_id "SURGE:TVS3301DRBR")
+		(lib_id "SURGE:TVS2701DRBR")
 		(at 116.84 81.28 0)
 		(unit 1)
@@
 			)
 		)
-		(property "Value" "TVS3301DRBR"
+		(property "Value" "TVS2701DRBR"
 			(at 125.73 87.6299 0)
 			(show_name no)
@@
 			)
 		)
-		(property "Datasheet" "https://www.ti.com/lit/ds/symlink/tvs3301.pdf"
+		(property "Datasheet" "http://www.ti.com/lit/ds/slvseq5a/slvseq5a.pdf"
 			(at 143.51 276.2 0)
 			(hide yes)
@@
 			)
 		)
-		(property "Field6" ""
-			(at 116.84 81.28 0)
+		(property "Height" "1"
+			(at 143.51 476.2 0)
 			(hide yes)
 			(show_name no)
@@
 					(size 1.27 1.27)
 				)
+				(justify left top)
 			)
 		)
-		(property "Field7" ""
-			(at 116.84 81.28 0)
+		(property "Mouser Part Number" "595-TVS2701DRBR"
+			(at 143.51 576.2 0)
 			(hide yes)
 			(show_name no)
@@
 					(size 1.27 1.27)
 				)
+				(justify left top)
 			)
 		)
-		(property "Part Description" ""
-			(at 116.84 81.28 0)
+		(property "Mouser Price/Stock" "https://www.mouser.co.uk/ProductDetail/Texas-Instruments/TVS2701DRBR?qs=byeeYqUIh0OuvTYsaTi%252BEg%3D%3D"
+			(at 143.51 676.2 0)
 			(hide yes)
 			(show_name no)
@@
 					(size 1.27 1.27)
 				)
+				(justify left top)
 			)
 		)
-		(property "Critical Parameter" ""
-			(at 116.84 81.28 0)
+		(property "Manufacturer_Name" "Texas Instruments"
+			(at 143.51 776.2 0)
 			(hide yes)
 			(show_name no)
@@
 					(size 1.27 1.27)
 				)
+				(justify left top)
 			)
 		)
-		(property "IRP,40K (A)" ""
-			(at 116.84 81.28 0)
+		(property "Manufacturer_Part_Number" "TVS2701DRBR"
+			(at 143.51 876.2 0)
 			(hide yes)
 			(show_name no)
@@
 					(size 1.27 1.27)
 				)
+				(justify left top)
 			)
 		)
-		(property "ISAT,10% (A)" ""
-			(at 116.84 81.28 0)
-			(hide yes)
-			(show_name no)
-			(do_not_autoplace no)
-			(effects
-				(font
-					(size 1.27 1.27)
-				)
-			)
-		)
-		(property "ISAT,30% (A)" ""
-			(at 116.84 81.28 0)
-			(hide yes)
-			(show_name no)
-			(do_not_autoplace no)
-			(effects
-				(font
-					(size 1.27 1.27)
-				)
-			)
-		)
-		(property "L (µH)" ""
-			(at 116.84 81.28 0)
-			(hide yes)
-			(show_name no)
-			(do_not_autoplace no)
-			(effects
-				(font
-					(size 1.27 1.27)
-				)
-			)
-		)
-		(property "Manufacturer" ""
-			(at 116.84 81.28 0)
-			(hide yes)
-			(show_name no)
-			(do_not_autoplace no)
-			(effects
-				(font
-					(size 1.27 1.27)
-				)
-			)
-		)
-		(property "Manufacturer URL" ""
-			(at 116.84 81.28 0)
-			(hide yes)
-			(show_name no)
-			(do_not_autoplace no)
-			(effects
-				(font
-					(size 1.27 1.27)
-				)
-			)
-		)
-		(property "Match Code" ""
-			(at 116.84 81.28 0)
-			(hide yes)
-			(show_name no)
-			(do_not_autoplace no)
-			(effects
-				(font
-					(size 1.27 1.27)
-				)
-			)
-		)
-		(property "Mounting Technology" ""
-			(at 116.84 81.28 0)
-			(hide yes)
-			(show_name no)
-			(do_not_autoplace no)
-			(effects
-				(font
-					(size 1.27 1.27)
-				)
-			)
-		)
-		(property "Part Number" ""
-			(at 116.84 81.28 0)
-			(hide yes)
-			(show_name no)
-			(do_not_autoplace no)
-			(effects
-				(font
-					(size 1.27 1.27)
-				)
-			)
-		)
-		(property "Published Date" ""
-			(at 116.84 81.28 0)
-			(hide yes)
-			(show_name no)
-			(do_not_autoplace no)
-			(effects
-				(font
-					(size 1.27 1.27)
-				)
-			)
-		)
-		(property "RDC max. (mΩ)" ""
-			(at 116.84 81.28 0)
-			(hide yes)
-			(show_name no)
-			(do_not_autoplace no)
-			(effects
-				(font
-					(size 1.27 1.27)
-				)
-			)
-		)
-		(property "RDC typ. (mΩ)" ""
-			(at 116.84 81.28 0)
-			(hide yes)
-			(show_name no)
-			(do_not_autoplace no)
-			(effects
-				(font
-					(size 1.27 1.27)
-				)
-			)
-		)
-		(property "Size" ""
-			(at 116.84 81.28 0)
-			(hide yes)
-			(show_name no)
-			(do_not_autoplace no)
-			(effects
-				(font
-					(size 1.27 1.27)
-				)
-			)
-		)
-		(property "Type/Size" ""
-			(at 116.84 81.28 0)
-			(hide yes)
-			(show_name no)
-			(do_not_autoplace no)
-			(effects
-				(font
-					(size 1.27 1.27)
-				)
-			)
-		)
-		(property "VOP (V)" ""
-			(at 116.84 81.28 0)
-			(hide yes)
-			(show_name no)
-			(do_not_autoplace no)
-			(effects
-				(font
-					(size 1.27 1.27)
-				)
-			)
-		)
-		(property "fres (MHz)" ""
-			(at 116.84 81.28 0)
-			(hide yes)
-			(show_name no)
-			(do_not_autoplace no)
-			(effects
-				(font
-					(size 1.27 1.27)
-				)
-			)
-		)

Commit message: 603 Unrouted
Parts:
- added C302: 1u, project_footprints:C_0402, symbol DEV:C_SMALL
- added R306: 47k, project_footprints:R_0402, symbol Device:R_Small
- added R307: 12k1, project_footprints:R_0402, symbol Device:R_Small
- added R308: 450k, project_footprints:R_0402, symbol Device:R_Small
- added R309, R310: 1k, project_footprints:R_0402, symbol DEV:R_SMALL
- added R311: 10k, project_footprints:R_0402, symbol DEV:R_SMALL
- added U303: ADS7128IRTER, project_footprints:QFN50P300X300X80-17N-D, symbol ADC:ADS7128IRTER
Connections:
- net +VIN: now also R308.2
- net GND: now also C302.2, R306.1, U303.17 (EP), U303.9 (GND)
- net RTN: now also R307.1
- net IMON: now reaches U302.18 (IMON)
- net IMON: now also R307.2, U303.16 (AIN1/GPIO1)
- new net +3V3: R309.1, R310.1, R311.1, U303.10 (DVDD), U303.7 (AVDD)
- new net DECAP: C302.1, U303.8 (DECAP)
- new net INT: R311.2, U303.12 (ALERT)
- new net SCL: R310.2, U303.13 (SCL)
- new net SDA: R309.2, U303.14 (SDA)
- new net VMON: R306.2, R308.1, U303.15 (AIN0/GPIO0)
- no-connect marks 5 -> 11
Other:
- note added: "Power Measuring ADC"
- moved on the sheet: C301, D301, J301, R301, R302, R303, R304, R305, U301, U302

Commit message: 400 Unrouted
Parts:
- added C303, C304: 1u, project_footprints:C_0402, symbol DEV:C_SMALL
Connections:
- net +3V3: now also C303.1, C304.1
- net GND: now also C303.2, C304.2
- net IMON: now also U303.1 (AIN2/GPIO2); no longer U303.16 (AIN1/GPIO1)
- net VMON: now also U303.16 (AIN1/GPIO1); no longer U303.15 (AIN0/GPIO0)
- net INT renamed ~{INT}

Commit message: 133 Unrouted
Parts:
- added C305: 47n, project_footprints:C_0402, symbol DEV:C_SMALL
- added TP301: 1.5mm, project_footprints:TestPoint_Pad_D1.5mm, symbol Connector:TestPoint_Small
Connections:
- net +VIN: now also TP301.1
- net RTN: now also C305.2
- net DVDT: now reaches U302.20 (DVDT)
- net DVDT: now also C305.1
- no-connect marks 11 -> 10
Other:
- moved on the sheet: C301, D301, J301, R301, R302, R303, U301
