File: pcbs/jabrj-control-v2/jabrj-control-v2.kicad_sch (KiCad schematic)
At the start: 11 parts

Commit message: 603 Unrouted
Other:
- sheet CM5 ports: added CAM_GPIO[0..2], I2C3{I2C}; removed CAM_GPIO[0..1]
- sheet Power ports: added {I2C}; removed none
Changed lines of the file:
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@@
 		)
 	)
+	(bus
+		(pts
+			(xy 96.52 106.68) (xy 121.92 106.68)
+		)
+		(stroke
+			(width 0)
+			(type default)
+		)
+	)
 	(polyline
 		(pts
@@
 	(wire
 		(pts
-			(xy 96.52 109.22) (xy 121.92 109.22)
+			(xy 96.52 111.76) (xy 121.92 111.76)
 		)
 		(stroke
@@
 		)
 		(pin "PCIE_PWR_EN" input
-			(at 96.52 109.22 0)
+			(at 96.52 111.76 0)
+			(effects
+				(font
+					(size 1.27 1.27)
+				)
+				(justify right)
+			)
+		)
+		(pin "{I2C}" bidirectional
+			(at 96.52 106.68 0)
 			(effects
 				(font
@@
 		)
 		(pin "PCIE_PWR_EN" output
-			(at 121.92 109.22 180)
+			(at 121.92 111.76 180)
 			(effects
 				(font
@@
 			)
 		)
-		(pin "CAM_GPIO[0..1]" bidirectional
+		(pin "CAM_GPIO[0..2]" bidirectional
 			(at 121.92 27.94 180)
 			(effects
 				(font
+					(size 1.27 1.27)
+				)
+				(justify left)
+			)
+		)
+		(pin "I2C3{I2C}" bidirectional
+			(at 121.92 106.68 180)
+			(effects
+				(font

Commit message: 400 Unrouted
Other:
- sheet CM5 ports: added UART2{UART}; removed none
- sheet CM5IO ports: added {UART}; removed none
Changed lines of the file:
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@@
 	(text "Can be broken off\nif IO isn't needed"
 		(exclude_from_sim no)
-		(at 58.42 81.28 0)
+		(at 58.42 77.47 0)
 		(effects
 			(font
@@
 	(bus
 		(pts
-			(xy 96.52 66.04) (xy 121.92 66.04)
+			(xy 96.52 71.12) (xy 121.92 71.12)
 		)
 		(stroke
@@
 	(bus
 		(pts
-			(xy 96.52 86.36) (xy 121.92 86.36)
+			(xy 96.52 81.28) (xy 121.92 81.28)
 		)
 		(stroke
@@
 	(bus
 		(pts
-			(xy 96.52 78.74) (xy 121.92 78.74)
+			(xy 96.52 66.04) (xy 121.92 66.04)
 		)
 		(stroke
@@
 	(bus
 		(pts
-			(xy 96.52 88.9) (xy 121.92 88.9)
+			(xy 96.52 83.82) (xy 121.92 83.82)
 		)
 		(stroke
@@
 	(bus
 		(pts
-			(xy 96.52 68.58) (xy 121.92 68.58)
+			(xy 96.52 73.66) (xy 121.92 73.66)
 		)
 		(stroke
@@
 	(wire
 		(pts
-			(xy 96.52 71.12) (xy 121.92 71.12)
+			(xy 96.52 76.2) (xy 121.92 76.2)
 		)
 		(stroke
@@
 		)
 	)
+	(bus
+		(pts
+			(xy 96.52 88.9) (xy 121.92 88.9)
+		)
+		(stroke
+			(width 0)
+			(type default)
+		)
+	)
 	(polyline
 		(pts
@@
 		)
 		(pin "ETH_LED[2..3]" output
-			(at 121.92 88.9 180)
+			(at 121.92 83.82 180)
 			(effects
 				(font
@@
 		)
 		(pin "ETH{MDI}" bidirectional
-			(at 121.92 86.36 180)
+			(at 121.92 81.28 180)
 			(effects
 				(font
@@
 		)
 		(pin "VBUS_EN" output
-			(at 121.92 71.12 180)
+			(at 121.92 76.2 180)
 			(effects
 				(font
@@
 		)
 		(pin "USB2_DEV{USB}" bidirectional
-			(at 121.92 78.74 180)
+			(at 121.92 66.04 180)
 			(effects
 				(font
@@
 		)
 		(pin "USB3_0{USB3}" bidirectional
-			(at 121.92 66.04 180)
+			(at 121.92 71.12 180)
 			(effects
 				(font
@@
 		)
 		(pin "USB3_1{USB3}" bidirectional
-			(at 121.92 68.58 180)
+			(at 121.92 73.66 180)
 			(effects
 				(font
@@
 			)
 		)
+		(pin "UART2{UART}" bidirectional
+			(at 121.92 88.9 180)
+			(effects
+				(font
+					(size 1.27 1.27)
+				)
+				(justify left)
+			)
+		)
 		(instances
 			(project "jabrj-control-v2"
@@
 		)
 		(pin "ETH_LED[2..3]" input
-			(at 96.52 88.9 0)
+			(at 96.52 83.82 0)
 			(effects
 				(font
@@
 		)
 		(pin "ETH{MDI}" bidirectional
-			(at 96.52 86.36 0)
+			(at 96.52 81.28 0)
 			(effects
 				(font
@@
 		)
 		(pin "USB{USB}" bidirectional
-			(at 96.52 78.74 0)
+			(at 96.52 66.04 0)
 			(effects
 				(font
@@
 		)
 		(pin "USB3_0{USB3}" bidirectional
-			(at 96.52 66.04 0)
+			(at 96.52 71.12 0)
 			(effects
 				(font
@@
 		)
 		(pin "USB3_1{USB3}" bidirectional
-			(at 96.52 68.58 0)
+			(at 96.52 73.66 0)
 			(effects
 				(font
@@
 		)
 		(pin "VBUS_EN" input
-			(at 96.52 71.12 0)
+			(at 96.52 76.2 0)
+			(effects
+				(font
+					(size 1.27 1.27)
+				)
+				(justify right)
+			)
+		)
+		(pin "{UART}" bidirectional
+			(at 96.52 88.9 0)
 			(effects
 				(font

Commit message: Updated all line endings
Parts:
- H101, H102, H104, H105: footprint Mounting_Wuerth:Mounting_Wuerth_WA-SMST-2.7mm_H1.5mm_9774015951 -> project_footprints:9774015951
Changed lines of the file:
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@@
 			)
 		)
-		(property "Footprint" "Mounting_Wuerth:Mounting_Wuerth_WA-SMST-2.7mm_H1.5mm_9774015951"
+		(property "Footprint" "project_footprints:9774015951"
 			(at 148.59 267.64 0)
 			(hide yes)
@@
 			)
 		)
-		(property "Footprint" "Mounting_Wuerth:Mounting_Wuerth_WA-SMST-2.7mm_H1.5mm_9774015951"
+		(property "Footprint" "project_footprints:9774015951"
 			(at 128.27 267.64 0)
 			(hide yes)
@@
 			)
 		)
-		(property "Footprint" "Mounting_Wuerth:Mounting_Wuerth_WA-SMST-2.7mm_H1.5mm_9774015951"
+		(property "Footprint" "project_footprints:9774015951"
 			(at 128.27 242.24 0)
 			(hide yes)
@@
 			)
 		)
-		(property "Footprint" "Mounting_Wuerth:Mounting_Wuerth_WA-SMST-2.7mm_H1.5mm_9774015951"
+		(property "Footprint" "project_footprints:9774015951"
 			(at 148.59 242.24 0)
 			(hide yes)
