File: pcbs/jabrj-control-v2/cm5.kicad_sch (KiCad schematic)
At the start: 24 parts, among them J702 JST-SH-4-Vertical, Q701 DMN21D2UFB-7B, SW701 TS20-42-25-WT-160-SMT-TR, U702 NX3DV221GM

Commit message: 133 Unrouted
Connections:
- net ~{OE} renamed ~{USB2_OE}
Changed lines of the file:
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@@
 		)
 	)
-	(label "~{OE}"
-		(at 223.52 73.66 0)
+	(label "~{USB2_OE}"
+		(at 220.98 73.66 0)
 		(effects
 			(font

Commit message: DRC Clean
Changed lines of the file:
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@@
+		)
+	)
+	(text_box "GPIO4 & GPIO5 can also be set to I2C2 instead if required."
+		(exclude_from_sim no)
+		(at 22.86 81.28 0)
+		(size 27.94 8.0376)
+		(margins 0.9525 0.9525 0.9525 0.9525)
+		(stroke
+			(width 0)
+			(type solid)
+		)
+		(fill
+			(type none)
+		)
+		(effects
+			(font
+				(size 1.27 1.27)
+			)
+			(justify left top)
 		)
 	)
